File: hardware/rs232.kicad_pcb (KiCad board)
At the start: 2 copper layers, 45 x 35 mm, 33 parts, among them J1 DB9, P1 CON-SENSOR, P2 CONN_5, P3 CONN_5, U1 M24C64, U2 SC16IS740, U3 SP3232EBCN, U4 DRILL, U5 DRILL, U6 DRILL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

Commit message: run drc
Other:
- board text added: "3.3V"
- board text removed: "3V3"
